File: paw-kbd/paw-kbd.kicad_pcb (KiCad board)
At the start: 2 copper layers, 131 x 80.7 mm, 63 parts, among them J1 OLED, J2 TRRS, J3 TRACKBALL, SW1 SW_PUSH, SW10 SW_PUSH, SW11 SW_PUSH, SW12 SW_PUSH, SW13 SW_PUSH, SW14 SW_PUSH, SW15 SW_PUSH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

Commit message: 2023-08-01 00:03:10
Parts:
- removed the D18 at (223.5, 100.0)
- removed U1: ProMicro, keeb-footprints:ProMicro_v2
- added D19: type="D" model="DIODE" lib="", kbd:D3_TH_SMD_v2, F.Cu at (248.0, 47.1)
- added D20: type="D" model="DIODE" lib="", kbd:D3_TH_SMD_v2, F.Cu at (248.0, 49.4)
- added SW20: SW_PUSH, keeb-footprints:ChocV1_V2_Hotswap_optional_reversed_choc_spacing, F.Cu at (137.9, 115.1)
- added U2: SeeeduinoXIAO, keeb-footprints:seed, F.Cu at (224.1, 36.3)
Connections:
- SW4 pad 1: ring -> SW19A
- SW5 pad 1: ring -> SW19A
- SW6 pad 1: ring -> SW19A
