File: paw-kbd/paw-kbd.kicad_sch (KiCad schematic)
At the start: 62 parts, among them J1 OLED, J2 TRRS, J3 TRACKBALL, SW1 SW_PUSH, SW10 SW_PUSH, SW11 SW_PUSH, SW12 SW_PUSH, SW13 SW_PUSH, SW14 SW_PUSH, SW15 SW_PUSH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

Commit message: seed
Parts:
- removed U1: ProMicro, keeb-footprints:ProMicro_v2, symbol kbd:ProMicro
- added U2: SeeeduinoXIAO, Seeeduino XIAO KICAD:Seeeduino XIAO-MOUDLE14P-2.54-21X17.8MM, symbol Seeeduino XIAO:SeeeduinoXIAO
Connections:
- net GND: now also U2.13 (GND)
- net SCL: now also U2.6 (PA9_A5_D5_SCL)
- net SDA: now also U2.5 (PA8_A4_D4_SDA)
- net VCC: now also U2.12 (3V3)
- net bottom: now also U2.9 (PA7_A8_D8_SCK)
- net far: now also U2.1 (PA02_A0_D0)
- net home: now also U2.10 (PA5_A9_D9_MISO)
- net index: now also U2.2 (PA4_A1_D1)
- net middle: now also U2.3 (PA10_A2_D2)
- net pinky: now also U2.7 (PB08_A6_D6_TX)
- net ring: now also U2.4 (PA11_A3_D3)
- net thumb: now also U2.8 (PB09_A7_D7_RX)
- net top: now also U2.11 (PA6_A10_D10_MOSI)

Commit message: 2023-08-01 00:03:10
Parts:
- added D19, D20: ${SIM.PARAMS}, kbd:D3_TH_SMD_v2, symbol Simulation_SPICE:DIODE
- added SW20: SW_PUSH, keeb-footprints:ChocV1_V2_Hotswap_optional_reversed_choc_spacing, symbol kbd:SW_PUSH
- U2: footprint Seeeduino XIAO KICAD:Seeeduino XIAO-MOUDLE14P-2.54-21X17.8MM -> keeb-footprints:seed
Connections:
- net ring is gone; now on net SW19A: SW4.1, SW5.1, SW6.1, U2.4 (PA11_A3_D3)
- net SW19B: now also D19.1 (A)
- net pinky: now also SW20.1
- net thumb: now also D19.2 (K), D20.2 (K)
- new net: D20.1 (A), SW20.2
Changed lines of the file:
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@@
   (junction (at 211.455 53.975) (diameter 0) (color 0 0 0 0)
   )
+  (junction (at 167.64 66.04) (diameter 0) (color 0 0 0 0)
+  )
   (junction (at 204.47 61.595) (diameter 0) (color 0 0 0 0)
   )
@@
   (junction (at 161.925 49.53) (diameter 0) (color 0 0 0 0)
   )
+  (junction (at 146.685 66.04) (diameter 0) (color 0 0 0 0)
+  )
+  (junction (at 161.925 85.725) (diameter 0) (color 0 0 0 0)
+  )
   (junction (at 233.68 66.04) (diameter 0) (color 0 0 0 0)
   )
@@
   (junction (at 204.47 85.725) (diameter 0) (color 0 0 0 0)
   )
+  (junction (at 182.88 85.725) (diameter 0) (color 0 0 0 0)
+  )
   (junction (at 211.455 66.04) (diameter 0) (color 0 0 0 0)
   )
@@
     (stroke (width 0) (type default))
   )
+  (wire (pts (xy 161.925 85.725) (xy 182.88 85.725))
+    (stroke (width 0) (type default))
+  )
   (wire (pts (xy 132.08 118.11) (xy 132.08 121.92))
     (stroke (width 0) (type default))
@@
     (stroke (width 0) (type default))
   )
+  (wire (pts (xy 182.88 85.725) (xy 204.47 85.725))
+    (stroke (width 0) (type default))
+  )
   (wire (pts (xy 192.405 107.95) (xy 203.835 107.95))
     (stroke (width 0) (type default))
@@
     (stroke (width 0) (type default))
   )
+  (wire (pts (xy 146.685 66.04) (xy 146.685 93.345))
+    (stroke (width 0) (type default))
+  )
   (wire (pts (xy 191.135 111.76) (xy 191.135 133.35))
     (stroke (width 0) (type default))
@@
     (stroke (width 0) (type default))
   )
-  (wire (pts (xy 143.51 85.725) (xy 204.47 85.725))
+  (wire (pts (xy 143.51 85.725) (xy 161.925 85.725))
     (stroke (width 0) (type default))
   )
@@
   )
   (wire (pts (xy 211.455 66.04) (xy 211.455 78.105))
+    (stroke (width 0) (type default))
+  )
+  (wire (pts (xy 167.64 66.04) (xy 167.64 99.695))
     (stroke (width 0) (type default))
   )
@@
     )
   )
+  (global_label "SW19B" (shape input) (at 182.88 93.345 0) (fields_autoplaced)
+    (effects (font (size 1.27 1.27)) (justify left))
+    (property "Intersheetrefs" "${INTERSHEET_REFS}" (at 192.2151 93.345 0)
+      (effects (font (size 1.27 1.27)) (justify left) hide)
+    )
+  )
   (global_label "SDA" (shape input) (at 266.7 114.3 270) (fields_autoplaced)
     (effects (font (size 1.524 1.524)) (justify right))
@@
     )
   )
+  (global_label "SW19A" (shape input) (at 167.64 99.695 0) (fields_autoplaced)
+    (effects (font (size 1.27 1.27)) (justify left))
+    (property "Intersheetrefs" "${INTERSHEET_REFS}" (at 176.7937 99.695 0)
+      (effects (font (size 1.27 1.27)) (justify left) hide)
+    )
+  )
   (symbol (lib_id "Simulation_SPICE:DIODE") (at 182.88 57.785 270) (unit 1)
     (in_bom yes) (on_board yes) (dnp no) (fields_autoplaced)
@@
     )
   )
+  (symbol (lib_id "Simulation_SPICE:DIODE") (at 161.925 89.535 90) (unit 1)
+    (in_bom yes) (on_board yes) (dnp no) (fields_autoplaced)
+    (property "Reference" "D20" (at 165.1 89.535 90)
+      (effects (font (size 1.27 1.27)) (justify right))
+    )
+    (property "Value" "${SIM.PARAMS}" (at 159.385 88.2651 90)
+      (effects (font (size 1.27 1.27)) (justify left) hide)
+    )
+    (property "Footprint" "kbd:D3_TH_SMD_v2" (at 161.925 89.535 0)
+      (effects (font (size 1.27 1.27)) hide)
+    )
+    (property "Datasheet" "~" (at 161.925 89.535 0)
+      (effects (font (size 1.27 1.27)) hide)
+    )
+    (property "Sim.Device" "SPICE" (at 161.925 89.535 0)
+      (effects (font (size 1.27 1.27)) (justify left) hide)
+    )
+    (property "Sim.Params" "type=\"D\" model=\"DIODE\" lib=\"\"" (at 410.845 171.45 0)
+      (effects (font (size 1.27 1.27)) hide)
+    )
+    (property "Sim.Pins" "1=1 2=2" (at 410.845 171.45 0)
+      (effects (font (size 1.27 1.27)) hide)
+    )
+    (pin "1")
+    (pin "2")
+    (instances
+      (project "paw-kbd"
+        (path "/7dd9dccd-9c0c-4b3b-807a-5d4c5c5409e0"
+          (reference "D20") (unit 1)
+        )
+      )
+    )
+  )
   (symbol (lib_id "corne-chocolate-rescue:Jumper_NO_Small-Device") (at 206.375 119.38 180) (unit 1)
     (in_bom yes) (on_board yes) (dnp no)
@@
         (path "/7dd9dccd-9c0c-4b3b-807a-5d4c5c5409e0"
           (reference "JP4") (unit 1)
+        )
+      )
+    )
+  )
+  (symbol (lib_id "kbd:SW_PUSH") (at 154.305 93.345 0) (unit 1)
+    (in_bom yes) (on_board yes) (dnp no)
+    (property "Reference" "SW20" (at 157.48 90.805 0)
+      (effects (font (size 1.27 1.27)))
+    )
+    (property "Value" "SW_PUSH" (at 154.305 95.25 0)
+      (effects (font (size 1.27 1.27)))
+    )
+    (property "Footprint" "keeb-footprints:ChocV1_V2_Hotswap_optional_reversed_choc_spacing" (at 154.305 93.345 0)
+      (effects (font (size 1.27 1.27)) hide)
+    )
+    (property "Datasheet" "" (at 154.305 93.345 0)
+      (effects (font (size 1.27 1.27)))
+    )
+    (pin "1")
+    (pin "2")
+    (instances
+      (project "paw-kbd"
+        (path "/7dd9dccd-9c0c-4b3b-807a-5d4c5c5409e0"
+          (reference "SW20") (unit 1)
         )
       )
@@
         (path "/7dd9dccd-9c0c-4b3b-807a-5d4c5c5409e0"
           (reference "SW2") (unit 1)
+        )
+      )
+    )
+  )
+  (symbol (lib_id "Simulation_SPICE:DIODE") (at 182.88 89.535 90) (unit 1)
+    (in_bom yes) (on_board yes) (dnp no) (fields_autoplaced)
+    (property "Reference" "D19" (at 186.055 89.535 90)
+      (effects (font (size 1.27 1.27)) (justify right))
+    )
+    (property "Value" "${SIM.PARAMS}" (at 180.34 88.2651 90)
+      (effects (font (size 1.27 1.27)) (justify left) hide)
+    )
+    (property "Footprint" "kbd:D3_TH_SMD_v2" (at 182.88 89.535 0)
+      (effects (font (size 1.27 1.27)) hide)
+    )
+    (property "Datasheet" "~" (at 182.88 89.535 0)
+      (effects (font (size 1.27 1.27)) hide)
+    )
+    (property "Sim.Device" "SPICE" (at 182.88 89.535 0)
+      (effects (font (size 1.27 1.27)) (justify left) hide)
+    )
+    (property "Sim.Params" "type=\"D\" model=\"DIODE\" lib=\"\"" (at 431.8 171.45 0)
+      (effects (font (size 1.27 1.27)) hide)
+    )
+    (property "Sim.Pins" "1=1 2=2" (at 431.8 171.45 0)
+      (effects (font (size 1.27 1.27)) hide)
+    )
+    (pin "1")
+    (pin "2")
+    (instances
+      (project "paw-kbd"
+        (path "/7dd9dccd-9c0c-4b3b-807a-5d4c5c5409e0"
+          (reference "D19") (unit 1)
         )
       )
@@
       (effects (font (size 1.27 1.27)) (justify left))
     )
-    (property "Footprint" "Seeeduino XIAO KICAD:Seeeduino XIAO-MOUDLE14P-2.54-21X17.8MM" (at 39.37 46.99 0)
-      (effects (font (size 1.27 1.27)) hide)
-    )
+    (property "Footprint" "keeb-footprints:seed" (at 39.37 46.99 0)
+      (effects (font (size 1.27 1.27)) hide)
+    )
