File: paw-kbd/paw-kbd.kicad_sch (KiCad schematic)
At the start: 65 parts, among them J1 OLED, J2 TRRS, J3 TRACKBALL, SW1 SW_PUSH, SW10 SW_PUSH, SW11 SW_PUSH, SW12 SW_PUSH, SW13 SW_PUSH, SW14 SW_PUSH, SW15 SW_PUSH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

Commit message: 2023-08-02 23:56:07
Parts:
- added U1: ProMicro_r, keeb-footprints:ProMicro_v2, symbol kbd:ProMicro_r
Connections:
- net GND: now also U1.23 (GND), U1.3 (GND), U1.4 (GND)
- net SCL: now also U1.6 (SCL/D0/3)
- net SDA: now also JP16.1 (A), U1.5 (SDA/D1/2); no longer JP16.2 (C)
- net VCC: now also U1.21 (VCC)
- net reset: now also U1.22 (RST)
- net at J2.R1: now also JP16.2 (C); no longer JP16.1 (A)
Other:
- moved on the sheet: JP16
